File: Batteryboard.sch (KiCad schematic (older format))
At the start: 76 parts, among them J1 Conn_01x02_Male, J2 Conn_01x03_Male, J3 Conn_01x02_Male, J4 Conn_01x02_Male, Q1 SI7617DN-T1-GE3, Q2 SI7617DN-T1-GE3, Q3 SI7617DN-T1-GE3, Q4 SIS412DN-T1-GE3, Q5 SIS412DN-T1-GE3, Q6 SIS412DN-T1-GE3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

Commit message: fixed an error with D1 footprint
Parts:
- D1: footprint Diode_SMD:D_0805_2012Metric -> Diode_SMD:D_SOD-323
Changed lines of the file:
@@
 F 0 "D1" H 6550 7284 50  0000 C CNN
 F 1 "D_Schottky" H 6550 7375 50  0000 C CNN
-F 2 "Diode_SMD:D_0805_2012Metric" H 6550 7500 50  0001 C CNN
+F 2 "Diode_SMD:D_SOD-323" H 6550 7500 50  0001 C CNN
 F 3 "~" H 6550 7500 50  0001 C CNN
 	1    6550 7500

Commit message: final touches before stefka, fixed a couple small things
Parts:
- L1: footprint Inductor_SMD:L_0603_1608Metric -> Inductor_SMD:L_Vishay_IHLP-2525
- R10/RT1, R9, R9/RT2: footprint Resistor_SMD:R_0805_2012Metric -> Resistor_SMD:R_0603_1608Metric
Changed lines of the file:
@@
 F 0 "R9/RT2" H 2668 6496 50  0000 L CNN
 F 1 "9.1kOhm" H 2668 6405 50  0000 L CNN
-F 2 "Resistor_SMD:R_0805_2012Metric" V 2640 6440 50  0001 C CNN
+F 2 "Resistor_SMD:R_0603_1608Metric" V 2640 6440 50  0001 C CNN
 F 3 "~" H 2600 6450 50  0001 C CNN
 	1    2600 6450
@@
 F 0 "R10/RT1" H 2668 6096 50  0000 L CNN
 F 1 "2.49kOhm" H 2668 6005 50  0000 L CNN
-F 2 "Resistor_SMD:R_0805_2012Metric" V 2640 6040 50  0001 C CNN
+F 2 "Resistor_SMD:R_0603_1608Metric" V 2640 6040 50  0001 C CNN
 F 3 "~" H 2600 6050 50  0001 C CNN
 	1    2600 6050
@@
 F 0 "L1" V 7990 6550 50  0000 C CNN
 F 1 "6.8uH" V 7899 6550 50  0000 C CNN
-F 2 "Inductor_SMD:L_0603_1608Metric" H 7800 6550 50  0001 C CNN
+F 2 "Inductor_SMD:L_Vishay_IHLP-2525" H 7800 6550 50  0001 C CNN
 F 3 "~" H 7800 6550 50  0001 C CNN
 	1    7800 6550
@@
 F 0 "R9" H 11018 7996 50  0000 L CNN
 F 1 "27kOhm" H 11018 7905 50  0000 L CNN
-F 2 "Resistor_SMD:R_0805_2012Metric" V 10990 7940 50  0001 C CNN
+F 2 "Resistor_SMD:R_0603_1608Metric" V 10990 7940 50  0001 C CNN
 F 3 "~" H 10950 7950 50  0001 C CNN
 	1    10950 7950

Commit message: fixed J2, wrong footprint
Parts:
- J2: footprint Connector_JST:JST_EH_B3B-EH-A_1x03_P2.50mm_Vertical -> Connector_JST:JST_XH_B3B-XH-AM_1x03_P2.50mm_Vertical
Changed lines of the file:
@@
 F 0 "J2" H 11308 5781 50  0000 C CNN
 F 1 "Conn_01x03_Male" H 11308 5690 50  0000 C CNN
-F 2 "Connector_JST:JST_EH_B3B-EH-A_1x03_P2.50mm_Vertical" H 11200 5500 50  0001 C CNN
+F 2 "Connector_JST:JST_XH_B3B-XH-AM_1x03_P2.50mm_Vertical" H 11200 5500 50  0001 C CNN
 F 3 "~" H 11200 5500 50  0001 C CNN
 	1    11200 5500

Commit message: needed to use a different cap, cause the value wasnt on digikey
Parts:
- CTTC1: value 43nF -> 47nF
Changed lines of the file:
@@
 P 3150 6400
 F 0 "CTTC1" H 3265 6446 50  0000 L CNN
-F 1 "43nF" H 3265 6355 50  0000 L CNN
+F 1 "47nF" H 3265 6355 50  0000 L CNN
 F 2 "Capacitor_SMD:C_1206_3216Metric" H 3150 6400 50  0001 C CNN
 F 3 "~" H 3150 6400 50  0001 C CNN

Commit message: fixed some footprints
Parts:
- CTTC1: footprint Capacitor_SMD:C_1206_3216Metric -> Capacitor_SMD:C_0603_1608Metric
- R10/RT1, R9/RT2: footprint Resistor_SMD:R_0603_1608Metric -> Resistor_SMD:R_0805_2012Metric
Changed lines of the file:
@@
 F 0 "R9/RT2" H 2668 6496 50  0000 L CNN
 F 1 "9.1kOhm" H 2668 6405 50  0000 L CNN
-F 2 "Resistor_SMD:R_0603_1608Metric" V 2640 6440 50  0001 C CNN
+F 2 "Resistor_SMD:R_0805_2012Metric" V 2640 6440 50  0001 C CNN
 F 3 "~" H 2600 6450 50  0001 C CNN
 	1    2600 6450
@@
 F 0 "R10/RT1" H 2668 6096 50  0000 L CNN
 F 1 "2.49kOhm" H 2668 6005 50  0000 L CNN
-F 2 "Resistor_SMD:R_0603_1608Metric" V 2640 6040 50  0001 C CNN
+F 2 "Resistor_SMD:R_0805_2012Metric" V 2640 6040 50  0001 C CNN
 F 3 "~" H 2600 6050 50  0001 C CNN
 	1    2600 6050
@@
 F 0 "CTTC1" H 3265 6446 50  0000 L CNN
 F 1 "47nF" H 3265 6355 50  0000 L CNN
-F 2 "Capacitor_SMD:C_1206_3216Metric" H 3150 6400 50  0001 C CNN
+F 2 "Capacitor_SMD:C_0603_1608Metric" H 3150 6400 50  0001 C CNN
 F 3 "~" H 3150 6400 50  0001 C CNN
 	1    3150 6400
